File: kicad_files/switch_footprints.kicad_sch (KiCad schematic)
At the start: 81 parts

Commit message: Update some components metadata up to RGB LEDs
Parts:
- HE1, HE10, HE11, HE12, HE13, HE14, HE15, HE16, HE17, HE18, HE19, HE2, HE20, HE21, HE22, HE23, HE24, HE25, HE26, HE27, HE28, HE29, HE3, HE30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: Manufacturer Kailh -> (none); Manufacturer Part Number CPG151101S11 -> (none)
