File: kicad_files/dcdc.kicad_sch (KiCad schematic)
At the start: 10 parts, among them U89 AP63203

Commit message: Pre-release modifications and checks
- Organize schematic, designators reset
- Remove empty "opamps" sheet
- Finish routing
- DRC ran, errors corrected
- Indicator cutout smoothened
Parts:
- renumbered C19 to C26, C20 to C27, C21 to C28, C22 to C29, R11 to R17, U89 to U90
Changed lines of the file:
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@@
 		(on_board yes)
 		(dnp no)
-		(property "Reference" "C20"
+		(property "Reference" "C27"
 			(at 504.19 436.8799 0)
 			(effects
@@
 			(project "M75H"
 				(path "/9ce6b20d-0a6c-402a-b232-5eafd6242eb3/314078ed-4566-47ce-b09f-b51d20fed207"
-					(reference "C20")
+					(reference "C27")
 					(unit 1)
 				)
@@
 		(dnp no)
 		(fields_autoplaced yes)
-		(property "Reference" "#PWR0176"
+		(property "Reference" "#PWR0195"
 			(at 606.425 429.26 0)
 			(effects
@@
 			(project "M75H"
 				(path "/9ce6b20d-0a6c-402a-b232-5eafd6242eb3/314078ed-4566-47ce-b09f-b51d20fed207"
-					(reference "#PWR0176")
+					(reference "#PWR0195")
 					(unit 1)
 				)
@@
 		(dnp no)
 		(fields_autoplaced yes)
-		(property "Reference" "R11"
+		(property "Reference" "R17"
 			(at 617.22 436.8799 0)
 			(effects
@@
 			(project "M75H"
 				(path "/9ce6b20d-0a6c-402a-b232-5eafd6242eb3/314078ed-4566-47ce-b09f-b51d20fed207"
-					(reference "R11")
+					(reference "R17")
 					(unit 1)
 				)
@@
 		(on_board yes)
 		(dnp no)
-		(property "Reference" "#PWR0177"
+		(property "Reference" "#PWR0196"
 			(at 508 450.85 0)
 			(effects
@@
 			(project "M75H"
 				(path "/9ce6b20d-0a6c-402a-b232-5eafd6242eb3/314078ed-4566-47ce-b09f-b51d20fed207"
-					(reference "#PWR0177")
+					(reference "#PWR0196")
 					(unit 1)
 				)
@@
 		(on_board yes)
 		(dnp no)
-		(property "Reference" "#PWR0181"
+		(property "Reference" "#PWR0200"
 			(at 587.375 462.28 0)
 			(effects
@@
 			(project "M75H"
 				(path "/9ce6b20d-0a6c-402a-b232-5eafd6242eb3/314078ed-4566-47ce-b09f-b51d20fed207"
-					(reference "#PWR0181")
+					(reference "#PWR0200")
 					(unit 1)
 				)
@@
 		(dnp no)
 		(fields_autoplaced yes)
-		(property "Reference" "U89"
+		(property "Reference" "U90"
 			(at 539.75 424.18 0)
 			(effects
@@
 			(project "M75H"
 				(path "/9ce6b20d-0a6c-402a-b232-5eafd6242eb3/314078ed-4566-47ce-b09f-b51d20fed207"
-					(reference "U89")
+					(reference "U90")
 					(unit 1)
 				)
@@
 		(on_board yes)
 		(dnp no)
-		(property "Reference" "#PWR0180"
+		(property "Reference" "#PWR0199"
 			(at 539.75 455.93 0)
 			(effects
@@
 			(project "M75H"
 				(path "/9ce6b20d-0a6c-402a-b232-5eafd6242eb3/314078ed-4566-47ce-b09f-b51d20fed207"
-					(reference "#PWR0180")
+					(reference "#PWR0199")
 					(unit 1)
 				)
@@
 		(on_board yes)
 		(dnp no)
-		(property "Reference" "C22"
+		(property "Reference" "C29"
 			(at 591.185 448.3099 0)
 			(effects
@@
 			(project "M75H"
 				(path "/9ce6b20d-0a6c-402a-b232-5eafd6242eb3/314078ed-4566-47ce-b09f-b51d20fed207"
-					(reference "C22")
+					(reference "C29")
 					(unit 1)
 				)
@@
 		(on_board yes)
 		(dnp no)
-		(property "Reference" "C21"
+		(property "Reference" "C28"
 			(at 602.615 439.4201 0)
 			(effects
@@
 			(project "M75H"
 				(path "/9ce6b20d-0a6c-402a-b232-5eafd6242eb3/314078ed-4566-47ce-b09f-b51d20fed207"
-					(reference "C21")
+					(reference "C28")
 					(unit 1)
 				)
@@
 		(on_board yes)
 		(dnp no)
-		(property "Reference" "#PWR0179"
+		(property "Reference" "#PWR0198"
 			(at 614.68 450.85 0)
 			(effects
@@
 			(project "M75H"
 				(path "/9ce6b20d-0a6c-402a-b232-5eafd6242eb3/314078ed-4566-47ce-b09f-b51d20fed207"
-					(reference "#PWR0179")
+					(reference "#PWR0198")
 					(unit 1)
 				)
@@
 		(on_board yes)
 		(dnp no)
-		(property "Reference" "C19"
+		(property "Reference" "C26"
 			(at 563.8799 427.99 0)
 			(effects
@@
 			(project "M75H"
 				(path "/9ce6b20d-0a6c-402a-b232-5eafd6242eb3/314078ed-4566-47ce-b09f-b51d20fed207"
-					(reference "C19")
+					(reference "C26")
 					(unit 1)
 				)
@@
 		(on_board yes)
 		(dnp no)
-		(property "Reference" "#PWR0178"
+		(property "Reference" "#PWR0197"
 			(at 606.425 450.85 0)
 			(effects
@@
 			(project "M75H"
 				(path "/9ce6b20d-0a6c-402a-b232-5eafd6242eb3/314078ed-4566-47ce-b09f-b51d20fed207"
-					(reference "#PWR0178")
-					(unit 1)
-				)
+					(reference "#PWR0197")
+					(unit 1)
+				)

Commit message: Update some components metadata up to RGB LEDs
Parts:
- C26, C28: Manufacturer (none) -> Guangdong Fenghua Advanced Tech; Manufacturer Part Number (none) -> 06035C104KAT2A; Vendor Part Number (none) -> LCSC C88476
- C27: Manufacturer (none) -> Murata; Manufacturer Part Number (none) -> GRM21BR61H106KE43L; Vendor Part Number (none) -> LCSC C440198
- C29: Manufacturer (none) -> Guangdong Fenghua Advanced Tech; Manufacturer Part Number (none) -> 0805X226M100NT; Vendor Part Number (none) -> LCSC C36255
Changed lines of the file:
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@@
 			)
 		)
-		(property "Manufacturer" ""
+		(property "Manufacturer" "Murata"
 			(at 508 438.15 0)
 			(effects
@@
 			)
 		)
-		(property "Manufacturer Part Number" ""
+		(property "Manufacturer Part Number" "GRM21BR61H106KE43L"
 			(at 508 438.15 0)
 			(effects
@@
 			)
 		)
-		(property "Vendor Part Number" ""
+		(property "Vendor Part Number" "LCSC C440198"
 			(at 508 438.15 0)
 			(effects
@@
 			)
 		)
-		(property "Manufacturer" ""
+		(property "Manufacturer" "Guangdong Fenghua Advanced Tech"
 			(at 587.375 449.58 0)
 			(effects
@@
 			)
 		)
-		(property "Manufacturer Part Number" ""
+		(property "Manufacturer Part Number" "0805X226M100NT"
 			(at 587.375 449.58 0)
 			(effects
@@
 			)
 		)
-		(property "Vendor Part Number" ""
+		(property "Vendor Part Number" "LCSC C36255"
 			(at 587.375 449.58 0)
 			(effects
@@
 			)
 		)
-		(property "Manufacturer" ""
+		(property "Manufacturer" "Guangdong Fenghua Advanced Tech"
 			(at 606.425 438.15 0)
 			(effects
@@
 			)
 		)
-		(property "Manufacturer Part Number" ""
+		(property "Manufacturer Part Number" "06035C104KAT2A"
 			(at 606.425 438.15 0)
 			(effects
@@
 			)
 		)
-		(property "Vendor Part Number" ""
+		(property "Vendor Part Number" "LCSC C88476"
 			(at 606.425 438.15 0)
 			(effects
@@
 			)
 		)
-		(property "Manufacturer" ""
+		(property "Manufacturer" "Guangdong Fenghua Advanced Tech"
 			(at 565.15 431.8 0)
 			(effects
@@
 			)
 		)
-		(property "Manufacturer Part Number" ""
+		(property "Manufacturer Part Number" "06035C104KAT2A"
 			(at 565.15 431.8 0)
 			(effects
@@
 			)
 		)
-		(property "Vendor Part Number" ""
+		(property "Vendor Part Number" "LCSC C88476"
 			(at 565.15 431.8 0)
 			(effects

Commit message: Finish adding metadata, release-ready
Parts:
- JP1, TP1, TP2: now left out of the parts list
- R17: Manufacturer (none) -> Uniroyal; Manufacturer Part Number (none) -> 0603WAF1003T5E; Vendor Part Number (none) -> LCSC C25803
Changed lines of the file:
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@@
 		(unit 1)
 		(exclude_from_sim no)
-		(in_bom yes)
+		(in_bom no)
 		(on_board yes)
 		(dnp no)
@@
 		(unit 1)
 		(exclude_from_sim no)
-		(in_bom yes)
+		(in_bom no)
 		(on_board yes)
 		(dnp no)
@@
 			)
 		)
-		(property "Manufacturer" ""
+		(property "Manufacturer" "Uniroyal"
 			(at 614.68 438.15 0)
 			(effects
@@
 			)
 		)
-		(property "Manufacturer Part Number" ""
+		(property "Manufacturer Part Number" "0603WAF1003T5E"
 			(at 614.68 438.15 0)
 			(effects
@@
 			)
 		)
-		(property "Vendor Part Number" ""
+		(property "Vendor Part Number" "LCSC C25803"
 			(at 614.68 438.15 0)
 			(effects
@@
 		(unit 1)
 		(exclude_from_sim yes)
-		(in_bom yes)
-		(on_board yes)
-		(dnp no)
+		(in_bom no)
+		(on_board yes)
+		(dnp no)
