File: kicad_files/sensors.kicad_sch (KiCad schematic)
At the start: 93 parts, among them U10 AH3503, U11 AH3503, U12 AH3503, U13 AH3503, U14 AH3503, U15 AH3503, U16 AH3503, U17 AH3503, U18 AH3503, U19 AH3503, U2 AH3503, U20 AH3503, U21 AH3503, U22 AH3503, U23 AH3503, U24 AH3503, U25 AH3503, U26 AH3503, U27 AH3503, U28 AH3503, U29 AH3503, U3 AH3503, U30 AH3503, U31 AH3503, U32 AH3503, U33 AH3503, U34 AH3503, U35 AH3503, U36 AH3503, U37 AH3503, U38 AH3503, U39 AH3503, U4 AH3503, U40 AH3503, U41 AH3503, U42 AH3503, U43 AH3503, U44 AH3503, U45 AH3503, U46 AH3503, U47 AH3503, U48 AH3503, U49 AH3503, U5 AH3503, U50 AH3503, U51 AH3503, U52 AH3503, U53 AH3503, U54 AH3503, U55 AH3503, U56 AH3503, U57 AH3503, U58 AH3503, U59 AH3503, U6 AH3503, U60 AH3503, U61 AH3503, U62 AH3503, U63 AH3503, U64 AH3503, U65 AH3503, U66 AH3503, U67 AH3503, U68 AH3503, U69 AH3503, U7 AH3503, U70 AH3503, U71 AH3503, U72 AH3503, U73 AH3503, U74 AH3503, U75 AH3503, U76 AH3503, U77 AH3503, U78 AH3503, U79 AH3503, U8 AH3503, U80 AH3503, U81 AH3503, U82 AH3503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

Commit message: Pre-release modifications and checks
- Organize schematic, designators reset
- Remove empty "opamps" sheet
- Finish routing
- DRC ran, errors corrected
- Indicator cutout smoothened
Parts:
- renumbered C13 to C20, C14 to C21, C15 to C22, C16 to C23, C17 to C24, C18 to C25, U9 to U10, U10 to U11, U11 to U12, U12 to U13, U13 to U14, U14 to U15, U15 to U16, U16 to U17, U17 to U18, U18 to U19, U19 to U20, U20 to U21, U21 to U22, U22 to U23, U23 to U24, U24 to U25, U25 to U26, U26 to U27, U27 to U28, U28 to U29, U2 to U3, U29 to U30, U30 to U31, U31 to U32, U32 to U33, U33 to U34, U34 to U35, U35 to U36, U36 to U37, U37 to U38, U38 to U39, U3 to U4, U39 to U40, U40 to U41, U41 to U42, U42 to U43, U43 to U44, U44 to U45, U45 to U46, U46 to U47, U47 to U48, U48 to U49, U4 to U5, U49 to U50, U50 to U51, U51 to U52, U52 to U53, U53 to U54, U54 to U55, U55 to U56, U56 to U57, U57 to U58, U58 to U59, U5 to U6, U59 to U60, U60 to U61, U61 to U62, U62 to U63, U63 to U64, U64 to U65, U65 to U66, U66 to U67, U67 to U68, U68 to U69, U6 to U7, U69 to U70, U70 to U71, U71 to U72, U72 to U73, U73 to U74, U74 to U75, U75 to U76, U76 to U77, U77 to U78, U78 to U79, U7 to U8, U79 to U80, U80 to U81, U81 to U82, U82 to U83, U83 to U84, U84 to U85, U85 to U86, U86 to U87, U87 to U88, U88 to U89, U8 to U9

Commit message: Update some components metadata up to RGB LEDs
Parts:
- C20, C21, C22, C23, C24, C25: Manufacturer Kyocera -> Guangdong Fenghua Advanced Tech
Changed lines of the file:
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@@
 			)
 		)
-		(property "Manufacturer" "Kyocera"
+		(property "Manufacturer" "Guangdong Fenghua Advanced Tech"
 			(at 371.475 352.425 0)
 			(effects
@@
 			)
 		)
-		(property "Manufacturer" "Kyocera"
+		(property "Manufacturer" "Guangdong Fenghua Advanced Tech"
 			(at 434.975 352.425 0)
 			(effects
@@
 			)
 		)
-		(property "Manufacturer" "Kyocera"
+		(property "Manufacturer" "Guangdong Fenghua Advanced Tech"
 			(at 307.975 354.965 0)
 			(effects
@@
 			)
 		)
-		(property "Manufacturer" "Kyocera"
+		(property "Manufacturer" "Guangdong Fenghua Advanced Tech"
 			(at 625.475 351.79 0)
 			(effects
@@
 			)
 		)
-		(property "Manufacturer" "Kyocera"
+		(property "Manufacturer" "Guangdong Fenghua Advanced Tech"
 			(at 561.975 352.425 0)
 			(effects
@@
 			)
 		)
-		(property "Manufacturer" "Kyocera"
+		(property "Manufacturer" "Guangdong Fenghua Advanced Tech"
 			(at 499.11 352.425 0)
 			(effects

Commit message: Finish adding metadata, release-ready
Parts:
- U10, U11, U12, U13, U14, U15, U16, U17, U18, U19, U20, U21, U22, U23, U24, U25, U26, U27, U28, U29, U3, U30, U31, U32, U33, U34, U35, U36, U37, U38, U39, U4, U40, U41, U42, U43, U44, U45, U46, U47, U48, U49, U5, U50, U51, U52, U53, U54, U55, U56, U57, U58, U59, U6, U60, U61, U62, U63, U64, U65, U66, U67, U68, U69, U7, U70, U71, U72, U73, U74, U75, U76, U77, U78, U79, U8, U80, U81, U82, U83, U9: value AH3503 -> HAL4904; Manufacturer (none) -> Hallwee; Manufacturer Part Number (none) -> HAL4904
- U84, U85, U86, U87, U88, U89: Manufacturer (none) -> Texas Instruments; Manufacturer Part Number (none) -> CD74HC4067M; Vendor Part Number (none) -> LCSC C496123
